File: CURSO_PCB_DRONE_R8/CURSO_PCB_DRONE.kicad_pcb (KiCad board)
At the start: 4 copper layers, 102 x 49 mm, 163 parts, among them J1 USB_B_Micro, J10 CONN_MOT_1, J11 CONN_MOT_3, J12 LIDAR, J13 CONN_STM32_I2C, J14 CONN_MOT_2, J15 CONN_MOT_4, J16 Conn_Coaxial, J17 XT-60, J2 SWD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

Commit message: Add files via upload
Routing:
- net Net-(D9-Pad2): track 0.45 -> 4.51 mm
- net Net-(D1-Pad2): track 0.44 -> 4.37 mm
